File: InternalPCBCase/TopPlate/Top Plate.kicad_pcb (KiCad board)
At the start: 2 copper layers, 137.8 x 92.6 mm, 0 parts

Commit message: V1.01 PCB and Plates incl Gerbers
Parts:
- added SCREW1: MountingHole_2.2mm_M2_DIN965, Mounting_Holes:MountingHole_2.2mm_M2_DIN965, F.Cu at (94.0, 72.2)
- added SCREW2: MountingHole_2.2mm_M2_DIN965, Mounting_Holes:MountingHole_2.2mm_M2_DIN965, F.Cu at (94.0, 110.3)
- added SCREW3: MountingHole_2.2mm_M2_DIN965, Mounting_Holes:MountingHole_2.2mm_M2_DIN965, F.Cu at (128.5, 68.8)
- added SCREW4: MountingHole_2.2mm_M2_DIN965, Mounting_Holes:MountingHole_2.2mm_M2_DIN965, F.Cu at (128.5, 106.8)
- added SCREW5: MountingHole_2.2mm_M2_DIN965, Mounting_Holes:MountingHole_2.2mm_M2_DIN965, F.Cu at (154.9, 68.8)
- added SCREW6: MountingHole_2.2mm_M2_DIN965, Mounting_Holes:MountingHole_2.2mm_M2_DIN965, F.Cu at (154.9, 106.8)
- added SCREW7: MountingHole_2.2mm_M2_DIN965, Mounting_Holes:MountingHole_2.2mm_M2_DIN965, F.Cu at (189.2, 72.2)
- added SCREW8: MountingHole_2.2mm_M2_DIN965, Mounting_Holes:MountingHole_2.2mm_M2_DIN965, F.Cu at (184.8, 109.2)
Changed lines of the file:
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@@
     (tracks 0)
     (zones 0)
-    (modules 0)
+    (modules 8)
     (nets 1)
   )
   (page A4)
   (layers
-    (0 F.Cu signal hide)
-    (31 B.Cu signal hide)
+    (0 F.Cu signal)
+    (31 B.Cu signal)
     (32 B.Adhes user)
     (33 F.Adhes user)
@@
     (uvia_drill 0.1)
   )
+  (module Mounting_Holes:MountingHole_2.2mm_M2_DIN965 (layer F.Cu)
+    (at 93.96 72.15)
+    (descr "Mounting Hole 2.2mm, no annular, M2, DIN965")
+    (tags "mounting hole 2.2mm no annular m2 din965")
+    (attr virtual)
+    (fp_text reference SCREW1 (at 0 -2.9) (layer F.SilkS) hide
+      (effects (font (size 1 1) (thickness 0.15)))
+    )
+    (fp_text value MountingHole_2.2mm_M2_DIN965 (at 0 2.9) (layer F.Fab) hide
+      (effects (font (size 1 1) (thickness 0.15)))
+    )
+    (fp_text user %R (at 0.3 0) (layer F.Fab)
+      (effects (font (size 1 1) (thickness 0.15)))
+    )
+    (fp_circle (center 0 0) (end 1.9 0) (layer Cmts.User) (width 0.15))
+    (fp_circle (center 0 0) (end 2.15 0) (layer F.CrtYd) (width 0.05))
+    (pad 1 np_thru_hole circle (at 0 0) (size 2.2 2.2) (drill 2.2) (layers *.Cu *.Mask))
+  )
+  (module Mounting_Holes:MountingHole_2.2mm_M2_DIN965 (layer F.Cu)
+    (at 93.96 110.35)
+    (descr "Mounting Hole 2.2mm, no annular, M2, DIN965")
+    (tags "mounting hole 2.2mm no annular m2 din965")
+    (attr virtual)
+    (fp_text reference SCREW2 (at 0 -2.9) (layer F.SilkS) hide
+      (effects (font (size 1 1) (thickness 0.15)))
+    )
+    (fp_text value MountingHole_2.2mm_M2_DIN965 (at 0 2.9) (layer F.Fab) hide
+      (effects (font (size 1 1) (thickness 0.15)))
+    )
+    (fp_text user %R (at 0.3 0) (layer F.Fab)
+      (effects (font (size 1 1) (thickness 0.15)))
+    )
+    (fp_circle (center 0 0) (end 1.9 0) (layer Cmts.User) (width 0.15))
+    (fp_circle (center 0 0) (end 2.15 0) (layer F.CrtYd) (width 0.05))
+    (pad 1 np_thru_hole circle (at 0 0) (size 2.2 2.2) (drill 2.2) (layers *.Cu *.Mask))
+  )
+  (module Mounting_Holes:MountingHole_2.2mm_M2_DIN965 (layer F.Cu)
+    (at 128.5 68.75)
+    (descr "Mounting Hole 2.2mm, no annular, M2, DIN965")
+    (tags "mounting hole 2.2mm no annular m2 din965")
+    (attr virtual)
+    (fp_text reference SCREW3 (at 0 -2.9) (layer F.SilkS) hide
+      (effects (font (size 1 1) (thickness 0.15)))
+    )
+    (fp_text value MountingHole_2.2mm_M2_DIN965 (at 0 2.9) (layer F.Fab) hide
+      (effects (font (size 1 1) (thickness 0.15)))
+    )
+    (fp_text user %R (at 0.3 0) (layer F.Fab)
+      (effects (font (size 1 1) (thickness 0.15)))
+    )
+    (fp_circle (center 0 0) (end 1.9 0) (layer Cmts.User) (width 0.15))
+    (fp_circle (center 0 0) (end 2.15 0) (layer F.CrtYd) (width 0.05))
+    (pad 1 np_thru_hole circle (at 0 0) (size 2.2 2.2) (drill 2.2) (layers *.Cu *.Mask))
+  )
+  (module Mounting_Holes:MountingHole_2.2mm_M2_DIN965 (layer F.Cu)
+    (at 128.5 106.85)
+    (descr "Mounting Hole 2.2mm, no annular, M2, DIN965")
+    (tags "mounting hole 2.2mm no annular m2 din965")
+    (attr virtual)
+    (fp_text reference SCREW4 (at 0 -2.9) (layer F.SilkS) hide
+      (effects (font (size 1 1) (thickness 0.15)))
+    )
+    (fp_text value MountingHole_2.2mm_M2_DIN965 (at 0 2.9) (layer F.Fab) hide
+      (effects (font (size 1 1) (thickness 0.15)))
+    )
+    (fp_text user %R (at 0.3 0) (layer F.Fab)
+      (effects (font (size 1 1) (thickness 0.15)))
+    )
+    (fp_circle (center 0 0) (end 1.9 0) (layer Cmts.User) (width 0.15))
+    (fp_circle (center 0 0) (end 2.15 0) (layer F.CrtYd) (width 0.05))
+    (pad 1 np_thru_hole circle (at 0 0) (size 2.2 2.2) (drill 2.2) (layers *.Cu *.Mask))
+  )
+  (module Mounting_Holes:MountingHole_2.2mm_M2_DIN965 (layer F.Cu)
+    (at 154.91 68.75)
+    (descr "Mounting Hole 2.2mm, no annular, M2, DIN965")
+    (tags "mounting hole 2.2mm no annular m2 din965")
+    (attr virtual)
+    (fp_text reference SCREW5 (at 0 -2.9) (layer F.SilkS) hide
+      (effects (font (size 1 1) (thickness 0.15)))
+    )
+    (fp_text value MountingHole_2.2mm_M2_DIN965 (at 0 2.9) (layer F.Fab) hide
+      (effects (font (size 1 1) (thickness 0.15)))
+    )
+    (fp_text user %R (at 0.3 0) (layer F.Fab)
+      (effects (font (size 1 1) (thickness 0.15)))
+    )
+    (fp_circle (center 0 0) (end 1.9 0) (layer Cmts.User) (width 0.15))
+    (fp_circle (center 0 0) (end 2.15 0) (layer F.CrtYd) (width 0.05))
+    (pad 1 np_thru_hole circle (at 0 0) (size 2.2 2.2) (drill 2.2) (layers *.Cu *.Mask))
+  )
+  (module Mounting_Holes:MountingHole_2.2mm_M2_DIN965 (layer F.Cu)
+    (at 154.91 106.85)
+    (descr "Mounting Hole 2.2mm, no annular, M2, DIN965")
+    (tags "mounting hole 2.2mm no annular m2 din965")
+    (attr virtual)
+    (fp_text reference SCREW6 (at 0 -2.9) (layer F.SilkS) hide
+      (effects (font (size 1 1) (thickness 0.15)))
+    )
+    (fp_text value MountingHole_2.2mm_M2_DIN965 (at 0 2.9) (layer F.Fab) hide
+      (effects (font (size 1 1) (thickness 0.15)))
+    )
+    (fp_text user %R (at 0.3 0) (layer F.Fab)
+      (effects (font (size 1 1) (thickness 0.15)))
+    )
+    (fp_circle (center 0 0) (end 1.9 0) (layer Cmts.User) (width 0.15))
+    (fp_circle (center 0 0) (end 2.15 0) (layer F.CrtYd) (width 0.05))
+    (pad 1 np_thru_hole circle (at 0 0) (size 2.2 2.2) (drill 2.2) (layers *.Cu *.Mask))
+  )
+  (module Mounting_Holes:MountingHole_2.2mm_M2_DIN965 (layer F.Cu)
+    (at 189.25 72.15)
+    (descr "Mounting Hole 2.2mm, no annular, M2, DIN965")
+    (tags "mounting hole 2.2mm no annular m2 din965")
+    (attr virtual)
+    (fp_text reference SCREW7 (at 0 -2.9) (layer F.SilkS) hide
+      (effects (font (size 1 1) (thickness 0.15)))
+    )
+    (fp_text value MountingHole_2.2mm_M2_DIN965 (at 0 2.9) (layer F.Fab) hide
+      (effects (font (size 1 1) (thickness 0.15)))
+    )
+    (fp_text user %R (at 0.3 0) (layer F.Fab)
+      (effects (font (size 1 1) (thickness 0.15)))
+    )
+    (fp_circle (center 0 0) (end 1.9 0) (layer Cmts.User) (width 0.15))
+    (fp_circle (center 0 0) (end 2.15 0) (layer F.CrtYd) (width 0.05))
+    (pad 1 np_thru_hole circle (at 0 0) (size 2.2 2.2) (drill 2.2) (layers *.Cu *.Mask))
+  )
+  (module Mounting_Holes:MountingHole_2.2mm_M2_DIN965 (layer F.Cu)
+    (at 184.78 109.22)
+    (descr "Mounting Hole 2.2mm, no annular, M2, DIN965")
+    (tags "mounting hole 2.2mm no annular m2 din965")
+    (attr virtual)
+    (fp_text reference SCREW8 (at 0 -2.9) (layer F.SilkS) hide
+      (effects (font (size 1 1) (thickness 0.15)))
+    )
+    (fp_text value MountingHole_2.2mm_M2_DIN965 (at 0 2.9) (layer F.Fab) hide
+      (effects (font (size 1 1) (thickness 0.15)))
+    )
+    (fp_text user %R (at 0.3 0) (layer F.Fab)
+      (effects (font (size 1 1) (thickness 0.15)))
+    )
+    (fp_circle (center 0 0) (end 1.9 0) (layer Cmts.User) (width 0.15))
+    (fp_circle (center 0 0) (end 2.15 0) (layer F.CrtYd) (width 0.05))
+    (pad 1 np_thru_hole circle (at 0 0) (size 2.2 2.2) (drill 2.2) (layers *.Cu *.Mask))
+  )
   (gr_text JLCJLCJLCJLC (at 103.23 72.39) (layer F.SilkS)
