File: PCB_Choc_LED/ErgoTravel.sch (KiCad schematic (older format))
At the start: 195 parts, among them J1 Conn_01x05, J10 Conn_01x01, J11 Conn_01x01, J12 Conn_01x01, J13 Conn_01x02, J14 Conn_01x02, J2 Audio-Jack-4, J3 Audio-Jack-4, J4 Conn_01x06, J5 Conn_01x01, J6 Conn_01x01, J7 Conn_01x01, J8 Conn_01x01, J9 Conn_01x01, K1 KEYSW, K10 KEYSW, K11 KEYSW, K12 KEYSW, K13 KEYSW, K14 KEYSW, K15 KEYSW, K16 KEYSW, K17 KEYSW, K18 KEYSW, K19 KEYSW, K2 KEYSW, K20 KEYSW, K21 KEYSW, K22 KEYSW, K23 KEYSW, K24 KEYSW, K26 KEYSW, K27 KEYSW, K28 KEYSW, K3 KEYSW, K4 KEYSW, K5 KEYSW, K6 KEYSW, K7 KEYSW, K8 KEYSW, K9 KEYSW, Q1 2N7002, Q2 2N7002, SW1 SW_PUSH, SW2 SW_PUSH, SW3 SW_SPDT, SW4 SW_SPDT, U1 ProMicro

Commit message: adding prototype for mids
Parts:
- Q1, Q2: value 2N7002 -> Si2302
- R3, R4, R6, R7: value 100R -> 0R
Other:
- note added: "All resistors are 2k2"
Changed lines of the file:
@@
 P 9200 5750
 F 0 "Q2" H 9405 5796 50  0000 L CNN
-F 1 "2N7002" H 9405 5705 50  0000 L CNN
+F 1 "Si2302" H 9405 5705 50  0000 L CNN
 F 2 "Package_TO_SOT_SMD:SOT-23" H 9400 5675 50  0001 L CIN
 F 3 "https://www.fairchildsemi.com/datasheets/2N/2N7002.pdf" H 9200 5750 50  0001 L CNN
@@
 P 7700 5750
 F 0 "Q1" H 7905 5796 50  0000 L CNN
-F 1 "2N7002" H 7905 5705 50  0000 L CNN
+F 1 "Si2302" H 7905 5705 50  0000 L CNN
 F 2 "Package_TO_SOT_SMD:SOT-23" H 7900 5675 50  0001 L CIN
 F 3 "https://www.fairchildsemi.com/datasheets/2N/2N7002.pdf" H 7700 5750 50  0001 L CNN
@@
 P 6650 4250
 F 0 "R3" V 6443 4250 50  0000 C CNN
-F 1 "100R" V 6534 4250 50  0000 C CNN
+F 1 "0R" V 6534 4250 50  0000 C CNN
 F 2 "Resistor_SMD:R_0805_2012Metric_Pad1.15x1.40mm_HandSolder" V 6580 4250 50  0001 C CNN
 F 3 "~" H 6650 4250 50  0001 C CNN
@@
 P 7350 4250
 F 0 "R6" V 7143 4250 50  0000 C CNN
-F 1 "100R" V 7234 4250 50  0000 C CNN
+F 1 "0R" V 7234 4250 50  0000 C CNN
 F 2 "Resistor_SMD:R_0805_2012Metric_Pad1.15x1.40mm_HandSolder" V 7280 4250 50  0001 C CNN
 F 3 "~" H 7350 4250 50  0001 C CNN
@@
 P 7350 4600
 F 0 "R7" V 7143 4600 50  0000 C CNN
-F 1 "100R" V 7234 4600 50  0000 C CNN
+F 1 "0R" V 7234 4600 50  0000 C CNN
 F 2 "Resistor_SMD:R_0805_2012Metric_Pad1.15x1.40mm_HandSolder" V 7280 4600 50  0001 C CNN
 F 3 "~" H 7350 4600 50  0001 C CNN
@@
 P 6650 4600
 F 0 "R4" V 6443 4600 50  0000 C CNN
-F 1 "100R" V 6534 4600 50  0000 C CNN
+F 1 "0R" V 6534 4600 50  0000 C CNN
 F 2 "Resistor_SMD:R_0805_2012Metric_Pad1.15x1.40mm_HandSolder" V 6580 4600 50  0001 C CNN
 F 3 "~" H 6650 4600 50  0001 C CNN
@@
 Wire Wire Line
 	13350 2700 13400 2700
+Text Notes 11600 5500 0    60   ~ 0
+All resistors are 2k2
 $EndSCHEMATC
