File: PCB/ErgoTravel.sch (KiCad schematic (older format))
At the start: 76 parts, among them J1 Conn_01x05, J10 Conn_01x01, J11 Conn_01x01, J12 Conn_01x01, J13 Conn_01x02, J14 Conn_01x02, J2 Audio-Jack-4, J3 Audio-Jack-4, J4 Conn_01x06, J5 Conn_01x01, J6 Conn_01x01, J7 Conn_01x01, J8 Conn_01x01, J9 Conn_01x01, K1 KEYSW, K10 KEYSW, K11 KEYSW, K12 KEYSW, K13 KEYSW, K14 KEYSW, K15 KEYSW, K16 KEYSW, K17 KEYSW, K18 KEYSW, K19 KEYSW, K2 KEYSW, K20 KEYSW, K21 KEYSW, K22 KEYSW, K23 KEYSW, K24 KEYSW, K25 KEYSW, K26 KEYSW, K27 KEYSW, K28 KEYSW, K3 KEYSW, K4 KEYSW, K5 KEYSW, K6 KEYSW, K7 KEYSW, K8 KEYSW, K9 KEYSW, SW1 SW_PUSH, SW2 SW_PUSH, U1 ProMicro

Commit message: last Kicad4.7 commit
Parts:
- added SW3, SW4: SW_SPDT, footprints:SPDT_C128955, symbol SW_SPDT
Connections:
- net RAW: now also SW3.2 (B), SW4.2 (B); no longer J14.2 (Pin_2)
- new net: J14.2 (Pin_2), SW3.1 (A), SW4.1 (A)
- no-connect marks 2 -> 4
Other:
- moved on the sheet: R1, R2
Changed lines of the file:
@@
 L R R1
 U 1 1 5A9D7565
-P 9700 4600
-F 0 "R1" V 9780 4600 50  0000 C CNN
-F 1 "4.7k" V 9700 4600 50  0000 C CNN
-F 2 "Resistors_THT:R_Axial_DIN0207_L6.3mm_D2.5mm_P10.16mm_Horizontal" V 9630 4600 50  0001 C CNN
-F 3 "" H 9700 4600 50  0001 C CNN
-	1    9700 4600
+P 9700 5950
+F 0 "R1" V 9780 5950 50  0000 C CNN
+F 1 "4.7k" V 9700 5950 50  0000 C CNN
+F 2 "Resistors_THT:R_Axial_DIN0207_L6.3mm_D2.5mm_P10.16mm_Horizontal" V 9630 5950 50  0001 C CNN
+F 3 "" H 9700 5950 50  0001 C CNN
+	1    9700 5950
 	1    0    0    -1
 $EndComp
@@
 L R R2
 U 1 1 5A9D77B4
-P 10300 4600
-F 0 "R2" V 10380 4600 50  0000 C CNN
-F 1 "4.7k" V 10300 4600 50  0000 C CNN
-F 2 "Resistors_THT:R_Axial_DIN0207_L6.3mm_D2.5mm_P10.16mm_Horizontal" V 10230 4600 50  0001 C CNN
-F 3 "" H 10300 4600 50  0001 C CNN
-	1    10300 4600
+P 10300 5950
+F 0 "R2" V 10380 5950 50  0000 C CNN
+F 1 "4.7k" V 10300 5950 50  0000 C CNN
+F 2 "Resistors_THT:R_Axial_DIN0207_L6.3mm_D2.5mm_P10.16mm_Horizontal" V 10230 5950 50  0001 C CNN
+F 3 "" H 10300 5950 50  0001 C CNN
+	1    10300 5950
 	1    0    0    -1
 $EndComp
@@
 L VCC #PWR010
 U 1 1 5A9D79AD
-P 9700 4250
-F 0 "#PWR010" H 9700 4100 50  0001 C CNN
-F 1 "VCC" H 9700 4400 50  0000 C CNN
-F 2 "" H 9700 4250 50  0001 C CNN
-F 3 "" H 9700 4250 50  0001 C CNN
-	1    9700 4250
+P 9700 5600
+F 0 "#PWR010" H 9700 5450 50  0001 C CNN
+F 1 "VCC" H 9700 5750 50  0000 C CNN
+F 2 "" H 9700 5600 50  0001 C CNN
+F 3 "" H 9700 5600 50  0001 C CNN
+	1    9700 5600
 	1    0    0    -1
 $EndComp
@@
 L VCC #PWR011
 U 1 1 5A9D7A72
-P 10300 4250
-F 0 "#PWR011" H 10300 4100 50  0001 C CNN
-F 1 "VCC" H 10300 4400 50  0000 C CNN
-F 2 "" H 10300 4250 50  0001 C CNN
-F 3 "" H 10300 4250 50  0001 C CNN
-	1    10300 4250
-	1    0    0    -1
-$EndComp
-Wire Wire Line
-	9700 4250 9700 4450
-Wire Wire Line
-	10300 4250 10300 4450
-Text GLabel 9550 4900 0    60   Input ~ 0
+P 10300 5600
+F 0 "#PWR011" H 10300 5450 50  0001 C CNN
+F 1 "VCC" H 10300 5750 50  0000 C CNN
+F 2 "" H 10300 5600 50  0001 C CNN
+F 3 "" H 10300 5600 50  0001 C CNN
+	1    10300 5600
+	1    0    0    -1
+$EndComp
+Wire Wire Line
+	9700 5600 9700 5800
+Wire Wire Line
+	10300 5600 10300 5800
+Text GLabel 9550 6250 0    60   Input ~ 0
 sda
-Text GLabel 10150 4900 0    60   Input ~ 0
+Text GLabel 10150 6250 0    60   Input ~ 0
 scl
 Wire Wire Line
-	9550 4900 9700 4900
-Wire Wire Line
-	9700 4900 9700 4750
-Wire Wire Line
-	10150 4900 10300 4900
-Wire Wire Line
-	10300 4900 10300 4750
+	9550 6250 9700 6250
+Wire Wire Line
+	9700 6250 9700 6100
+Wire Wire Line
+	10150 6250 10300 6250
+Wire Wire Line
+	10300 6250 10300 6100
 NoConn ~ 2750 6100
 Wire Wire Line
@@
 RAW
 Wire Wire Line
-	9850 3350 9850 3550
-Text Label 9850 3550 0    60   ~ 0
-RAW
+	9850 3350 9850 4550
 $Comp
 L GND #PWR016
@@
 Wire Wire Line
 	9750 3450 9750 3350
+$Comp
+L SW_SPDT SW4
+U 1 1 5B52C4A2
+P 9550 4100
+F 0 "SW4" H 9550 4270 50  0000 C CNN
+F 1 "SW_SPDT" H 9550 3900 50  0000 C CNN
+F 2 "footprints:SPDT_C128955" H 9550 4100 50  0001 C CNN
+F 3 "" H 9550 4100 50  0001 C CNN
+	1    9550 4100
+	1    0    0    -1
+$EndComp
+$Comp
+L SW_SPDT SW3
+U 1 1 5B52C5A5
+P 9500 4650
+F 0 "SW3" H 9500 4820 50  0000 C CNN
+F 1 "SW_SPDT" H 9500 4450 50  0000 C CNN
+F 2 "footprints:SPDT_C128955" H 9500 4650 50  0001 C CNN
+F 3 "" H 9500 4650 50  0001 C CNN
+	1    9500 4650
+	1    0    0    -1
+$EndComp
+Wire Wire Line
+	9350 4100 9100 4100
+Wire Wire Line
+	9100 4100 9100 4650
+Wire Wire Line
+	9100 4350 8850 4350
+Wire Wire Line
+	9100 4650 9300 4650
+Connection ~ 9100 4350
+Text Label 8850 4350 0    60   ~ 0
+RAW
+Wire Wire Line
+	9850 4000 9750 4000
+Wire Wire Line
+	9850 4550 9700 4550
+Connection ~ 9850 4000
+NoConn ~ 9750 4200
+NoConn ~ 9700 4750
 $EndSCHEMATC

Commit message: added MX version (V1.1) to avoid extra JLCPCB fees
Parts:
- added H1: MountingHole, keyswitches:Stabilizer_MX_2u, symbol Mechanical:MountingHole
- D1, D10, D11, D12, D13, D14, D15, D16, D17, D18, D19, D2, D20, D21, D22, D23, D24, D25, D26, D27, D28, D3, D4, D5, D6, D7, D8, D9: symbol D -> ErgoTravel-rescue:D
- J1: symbol Conn_01x05 -> ErgoTravel-rescue:Conn_01x05
- J10, J11, J12, J5, J6, J7, J8, J9: symbol Conn_01x01 -> ErgoTravel-rescue:Conn_01x01
- J13, J14: symbol Conn_01x02 -> ErgoTravel-rescue:Conn_01x02
- J2, J3: symbol Audio-Jack-4 -> ErgoTravel-rescue:Audio-Jack-4
- J4: symbol Conn_01x06 -> ErgoTravel-rescue:Conn_01x06
- K1, K10, K11, K12, K13, K14, K15, K16, K17, K18, K19, K2, K20, K21, K22, K23, K24, K26, K27, K28, K3, K4, K5, K6, K7, K8, K9: footprint footprints:Mx_Alps_100-dualside -> keyswitches:SW_MX_reversible; symbol KEYSW -> ErgoTravel-rescue:KEYSW
- K25: footprint footprints:Mx_Alps_200-dualside -> keyswitches:SW_MX_reversible; symbol KEYSW -> ErgoTravel-rescue:KEYSW
- R1, R2: symbol R -> ErgoTravel-rescue:R
- SJ1: symbol SOLDER_JUMPER -> ErgoTravel-rescue:SOLDER_JUMPER
- SW1, SW2: symbol SW_PUSH -> ErgoTravel-rescue:SW_PUSH
- SW3, SW4: symbol SW_SPDT -> ErgoTravel-rescue:SW_SPDT
- U1: symbol ProMicro -> ErgoTravel-rescue:ProMicro
